File: 18_Mesure_Courant.sch (KiCad schematic (older format))
At the start: 13 parts, among them J1 Conn_01x01, J2 Conn_01x01, J3 Conn_01x01, J4 Conn_01x01, J5 Conn_01x01, J6 Conn_01x01, J7 Conn_01x01, U1 ACS712xLCTR-20A

Commit message: maj split librairies
Parts:
- J1, J2, J3, J4, J5, J6, J7: footprint Chimere:Castellated_conn -> Chimere_mods:Castellated_conn
Changed lines of the file:
@@
 F 0 "J3" H 4255 1317 50  0000 L CNN
 F 1 "Conn_01x01" H 4255 1226 50  0000 L CNN
-F 2 "Chimere:Castellated_conn" H 4175 1275 50  0001 C CNN
+F 2 "Chimere_mods:Castellated_conn" H 4175 1275 50  0001 C CNN
 F 3 "~" H 4175 1275 50  0001 C CNN
 	1    4175 1275
@@
 F 0 "J1" H 4255 967 50  0000 L CNN
 F 1 "Conn_01x01" H 4255 876 50  0000 L CNN
-F 2 "Chimere:Castellated_conn" H 4175 925 50  0001 C CNN
+F 2 "Chimere_mods:Castellated_conn" H 4175 925 50  0001 C CNN
 F 3 "~" H 4175 925 50  0001 C CNN
 	1    4175 925
@@
 F 0 "J6" H 4255 2017 50  0000 L CNN
 F 1 "Conn_01x01" H 4255 1926 50  0000 L CNN
-F 2 "Chimere:Castellated_conn" H 4175 1975 50  0001 C CNN
+F 2 "Chimere_mods:Castellated_conn" H 4175 1975 50  0001 C CNN
 F 3 "~" H 4175 1975 50  0001 C CNN
 	1    4175 1975
@@
 F 0 "J2" H 4255 1142 50  0000 L CNN
 F 1 "Conn_01x01" H 4255 1051 50  0000 L CNN
-F 2 "Chimere:Castellated_conn" H 4175 1100 50  0001 C CNN
+F 2 "Chimere_mods:Castellated_conn" H 4175 1100 50  0001 C CNN
 F 3 "~" H 4175 1100 50  0001 C CNN
 	1    4175 1100
@@
 F 0 "J7" H 4255 2192 50  0000 L CNN
 F 1 "Conn_01x01" H 4255 2101 50  0000 L CNN
-F 2 "Chimere:Castellated_conn" H 4175 2150 50  0001 C CNN
+F 2 "Chimere_mods:Castellated_conn" H 4175 2150 50  0001 C CNN
 F 3 "~" H 4175 2150 50  0001 C CNN
 	1    4175 2150
@@
 F 0 "J4" H 4255 1667 50  0000 L CNN
 F 1 "Conn_01x01" H 4255 1576 50  0000 L CNN
-F 2 "Chimere:Castellated_conn" H 4175 1625 50  0001 C CNN
+F 2 "Chimere_mods:Castellated_conn" H 4175 1625 50  0001 C CNN
 F 3 "~" H 4175 1625 50  0001 C CNN
 	1    4175 1625
@@
 F 0 "J5" H 4255 1842 50  0000 L CNN
 F 1 "Conn_01x01" H 4255 1751 50  0000 L CNN
-F 2 "Chimere:Castellated_conn" H 4175 1800 50  0001 C CNN
+F 2 "Chimere_mods:Castellated_conn" H 4175 1800 50  0001 C CNN
 F 3 "~" H 4175 1800 50  0001 C CNN
 	1    4175 1800
