File: 18_Mesure_Courant.kicad_sch (KiCad schematic)
At the start: 13 parts

Commit message: maj schéma
symboles depuis librairies
vérification empreintes
ajout ligne LCSC
Parts:
- removed ?: 100nF, Capacitor_SMD:C_0603_1608Metric, symbol Device:C
- added C3: 50V 100nF X7R ±10%, Capacitor_SMD:C_0603_1608Metric, symbol Device:C
- C1: renamed from ?; value 100nF -> 50V 100nF X7R ±10%; LCSC (none) -> C14663
- C2: renamed from ?; value 10uF -> 50V 10uF X7R ±10%; LCSC (none) -> C337485
- C4: renamed from ?; value 1nF -> 50V 1nF X7R ±10%; LCSC (none) -> C1588
- R1: renamed from ?; footprint Resistor_SMD:R_0603_1608Metric_Pad1.05x0.95mm_HandSolder -> Resistor_SMD:R_0603_1608Metric
- U1: renamed from ?; LCSC (none) -> C10681
- gave numbers to parts that had none: 7
Connections:
- net GND: now also C3.2
- net I_mes: now also C3.1
Other:
- note added: "ACS712ELCTR-20A-T C10681 SOIC-8_3.9x4.9x1.27P ACS712xLCTR-20A Package_SO:SOIC-8_3.9x4.9mm_P1.27mm"
- note added: "Chimere_mods:Castellated_conn"
- note removed: "ACS712ELCTR-20A-T C10681 SOIC-8_3.9x4.9x1.27P"

Commit message: maj config gerbers
génération des fichiers pour fabrication
ajout ref lcsc pour R1
Parts:
- R1: LCSC (none) -> C21190
Changed lines of the file:
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@@
+      (effects (font (size 1.27 1.27)) hide)
+    )
+    (property "LCSC" "C21190" (id 4) (at 109.22 95.25 90)
       (effects (font (size 1.27 1.27)) hide)
     )
